File: RoyalBlue54L-Feather.kicad_pcb (KiCad board)
At the start: 8 copper layers, 58.4 x 22.9 mm, 69 parts, among them J1 Conn_01x16_Pin, J2 Conn_01x12_Pin, J3 USB_C_Receptacle_USB2.0_16P, J4 Conn_01x02_MountingPin, J5 Conn_01x04_MountingPin, J6 Conn_01x05_MountingPin, J8 Conn_ARM_SWD_TagConnect_TC203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, SW1 SW_Push, SW2 SW_Push, U1 BM15x, U2 nPM1300-QEXX, U3 TPD3E001DRLR, U4 W25Q16JVUXIQ, U5 nRF52833-QDXX, U6 TXB0106RGY, Y1 32.768KHz, Y2 32MHz

Commit message: Fix the Feather's ERC and DRC findings, without changing its rules
Modified Source of the RoyalBlue54L Feather by Helmut Lord (Lord's Boards),
under CERN-OHL-P v2, from 9177387. Made on 25 September 2026 by an AI agent
(Claude, by Anthropic) through the Eloom CLI, for Matrice Technologies.
CHANGES.md is the licence's modification notice and lists every change.

- PWR_FLAG on five externally fed nets (5 power_pin_not_driven errors)
- TP7 moved 0.049 mm onto the 1.27 mm grid (4 endpoint_off_grid warnings)
- four short reroutes for hole clearance (5 hole_clearance errors)
- courtyards: TP5-TP12 on 1.0 mm pads at the same pitch, J5 moved 0.32 mm,
  J3 and J5 courtyards drawn to their outlines, J2 on the back like J1 with a
  mirrored footprint and identical copper (11 courtyards_overlap errors)
- the design's own embedded symbols and footprints archived verbatim into
  project libraries; nothing updated from KiCad 10's libraries
- silkscreen nudges: the "+" mark, LOGO1, R5 and C9

The project file, with the author's rules and exclusions, is 9177387's byte
for byte. ERC 43 -> 0 and DRC 62 -> 0 with schematic parity, KiCad 10.0.6;
the final runs are under runs/. The author has not reviewed these changes,
and passing ERC and DRC does not prove the board works.

Co-Authored-By: Claude Opus 5.5 <noreply@anthropic.com>
Parts:
- C1, C10, C12, C13, C14, C15, C16, C17, C18, C19, C20, C21, C22, C23, C24, C25, C7, C9: footprint Capacitor_SMD:C_0402_1005Metric -> RoyalBlue54L-Feather:C_0402_1005Metric
- C11, C2, C3, C4, C5, C6, C8: footprint Capacitor_SMD:C_0603_1608Metric -> RoyalBlue54L-Feather:C_0603_1608Metric
- D1: footprint LED_SMD:LED_0603_1608Metric -> RoyalBlue54L-Feather:LED_0603_1608Metric
- J2: footprint RoyalBlue54L-Feather-Connector_PinHeader_2.54mm:PinHeader_1x12_P2.54mm_Vertical -> RoyalBlue54L-Feather-Connector_PinHeader_2.54mm:PinHeader_1x12_P2.54mm_Vertical_Mirrored; moved to B.Cu
- J3: footprint marbastlib-various:USB_C_Receptacle_HRO_TYPE-C-31-M-12 -> RoyalBlue54L-Feather:USB_C_Receptacle_HRO_TYPE-C-31-M-12_ChamferedCourtyard
- J4: footprint Connector_JST:JST_PH_S2B-PH-SM4-TB_1x02-1MP_P2.00mm_Horizontal -> RoyalBlue54L-Feather:JST_PH_S2B-PH-SM4-TB_1x02-1MP_P2.00mm_Horizontal
- L1: footprint Inductor_SMD:L_0603_1608Metric -> RoyalBlue54L-Feather:L_0603_1608Metric
- R1, R4, R5, R6, R7, R8: footprint Resistor_SMD:R_0402_1005Metric -> RoyalBlue54L-Feather:R_0402_1005Metric
- TP10, TP11, TP12, TP5, TP6, TP7, TP8, TP9: footprint TestPoint:TestPoint_Pad_D1.5mm -> TestPoint:TestPoint_Pad_D1.0mm
- U1: footprint nordic-lib-kicad-nrf54-modules:BM15x-LGA-45_15.8x10mm -> RoyalBlue54L-Feather:BM15x-LGA-45_15.8x10mm
- U2: footprint Package_DFN_QFN:QFN-32-1EP_5x5mm_P0.5mm_EP3.6x3.6mm_ThermalVias -> RoyalBlue54L-Feather:QFN-32-1EP_5x5mm_P0.5mm_EP3.6x3.6mm_ThermalVias
- U3: footprint Package_TO_SOT_SMD:SOT-553 -> RoyalBlue54L-Feather:SOT-553
- U4: footprint Package_SON:Winbond_USON-8-1EP_3x2mm_P0.5mm_EP0.2x1.6mm -> RoyalBlue54L-Feather:Winbond_USON-8-1EP_3x2mm_P0.5mm_EP0.2x1.6mm
- U5: footprint Package_DFN_QFN:QFN-40-1EP_5x5mm_P0.4mm_EP3.6x3.6mm_ThermalVias -> RoyalBlue54L-Feather:QFN-40-1EP_5x5mm_P0.4mm_EP3.6x3.6mm_ThermalVias
- Y2: footprint Crystal:Crystal_SMD_2016-4Pin_2.0x1.6mm -> RoyalBlue54L-Feather:Crystal_SMD_2016-4Pin_2.0x1.6mm
- moved LOGO1 0.95 mm to (130.2, 102.8)
- moved J5 0.32 mm to (128.3, 96.6)
- turned J2 to -90 degrees
