File: sch/Connectors.kicad_sch (KiCad schematic)
At the start: 4 parts, among them J1 Conn_01x16_Pin, J2 Conn_01x12_Pin, J4 Conn_01x02_MountingPin, J5 Conn_01x04_MountingPin

Commit message: Fix the Feather's ERC and DRC findings, without changing its rules
Modified Source of the RoyalBlue54L Feather by Helmut Lord (Lord's Boards),
under CERN-OHL-P v2, from 9177387. Made on 25 September 2026 by an AI agent
(Claude, by Anthropic) through the Eloom CLI, for Matrice Technologies.
CHANGES.md is the licence's modification notice and lists every change.

- PWR_FLAG on five externally fed nets (5 power_pin_not_driven errors)
- TP7 moved 0.049 mm onto the 1.27 mm grid (4 endpoint_off_grid warnings)
- four short reroutes for hole clearance (5 hole_clearance errors)
- courtyards: TP5-TP12 on 1.0 mm pads at the same pitch, J5 moved 0.32 mm,
  J3 and J5 courtyards drawn to their outlines, J2 on the back like J1 with a
  mirrored footprint and identical copper (11 courtyards_overlap errors)
- the design's own embedded symbols and footprints archived verbatim into
  project libraries; nothing updated from KiCad 10's libraries
- silkscreen nudges: the "+" mark, LOGO1, R5 and C9

The project file, with the author's rules and exclusions, is 9177387's byte
for byte. ERC 43 -> 0 and DRC 62 -> 0 with schematic parity, KiCad 10.0.6;
the final runs are under runs/. The author has not reviewed these changes,
and passing ERC and DRC does not prove the board works.

Co-Authored-By: Claude Opus 5.5 <noreply@anthropic.com>
Parts:
- J2: footprint RoyalBlue54L-Feather-Connector_PinHeader_2.54mm:PinHeader_1x12_P2.54mm_Vertical -> RoyalBlue54L-Feather-Connector_PinHeader_2.54mm:PinHeader_1x12_P2.54mm_Vertical_Mirrored
- J4: footprint Connector_JST:JST_PH_S2B-PH-SM4-TB_1x02-1MP_P2.00mm_Horizontal -> RoyalBlue54L-Feather:JST_PH_S2B-PH-SM4-TB_1x02-1MP_P2.00mm_Horizontal
Changed lines of the file:
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@@
+		(color 0 0 0 0)
+	)
+	(junction
+		(at 186.69 99.06)
+		(diameter 0)
+		(color 0 0 0 0)
+	)
+	(junction
+		(at 181.61 106.68)
+		(diameter 0)
 		(color 0 0 0 0)
 	)
@@
 	(wire
 		(pts
-			(xy 181.61 99.06) (xy 191.77 99.06)
+			(xy 181.61 99.06) (xy 186.69 99.06)
+		)
+		(stroke
+			(width 0)
+			(type default)
+		)
+	)
+	(wire
+		(pts
+			(xy 186.69 99.06) (xy 191.77 99.06)
 		)
 		(stroke
@@
 			)
 		)
-		(property "Footprint" "RoyalBlue54L-Feather-Connector_PinHeader_2.54mm:PinHeader_1x12_P2.54mm_Vertical"
+		(property "Footprint" "RoyalBlue54L-Feather-Connector_PinHeader_2.54mm:PinHeader_1x12_P2.54mm_Vertical_Mirrored"
 			(at 115.57 101.6 0)
 			(effects
@@
 			)
 		)
-		(property "Footprint" "Connector_JST:JST_PH_S2B-PH-SM4-TB_1x02-1MP_P2.00mm_Horizontal"
+		(property "Footprint" "RoyalBlue54L-Feather:JST_PH_S2B-PH-SM4-TB_1x02-1MP_P2.00mm_Horizontal"
 			(at 176.53 99.06 0)
 			(effects
@@
 					(unit 1)
 				)
+			)
+		)
+	)
+	(symbol
+		(lib_id "power:PWR_FLAG")
+		(at 186.69 99.06 180)
+		(unit 1)
+		(exclude_from_sim no)
+		(in_bom yes)
+		(on_board yes)
+		(dnp no)
+		(property "Reference" "#FLG04"
+			(at 186.69 100.965 0)
+			(effects
+				(font
+					(size 1.27 1.27)
+				)
+				(hide yes)
+			)
+		)
+		(property "Value" "PWR_FLAG"
+			(at 186.69 102.87 0)
+			(effects
+				(font
+					(size 1.27 1.27)
+				)
+			)
+		)
+		(property "Footprint" ""
+			(at 186.69 99.06 0)
+			(effects
+				(font
+					(size 1.27 1.27)
+				)
+				(hide yes)
+			)
+		)
+		(property "Datasheet" ""
+			(at 186.69 99.06 0)
+			(effects
+				(font
+					(size 1.27 1.27)
+				)
+				(hide yes)
+			)
+		)
+		(property "Description" "Special symbol for telling ERC where power comes from"
+			(at 186.69 99.06 0)
+			(effects
+				(font
+					(size 1.27 1.27)
+				)
+				(hide yes)
+			)
+		)
+		(pin "1"
+		)
+		(instances
+			(project "RoyalBlue54L-Feather"
+				(path "/ba76ff89-c129-45ae-a3c9-97538370856c/0a43c989-a862-4ff1-8fb5-5f7c93f777a1"
+					(reference "#FLG04")
+					(unit 1)
+				)
+			)
+		)
+	)
+	(symbol
+		(lib_id "power:PWR_FLAG")
+		(at 181.61 106.68 180)
+		(unit 1)
+		(exclude_from_sim no)
+		(in_bom yes)
+		(on_board yes)
+		(dnp no)
+		(property "Reference" "#FLG05"
+			(at 181.61 108.585 0)
+			(effects
+				(font
+					(size 1.27 1.27)
+				)
+				(hide yes)
+			)
+		)
+		(property "Value" "PWR_FLAG"
+			(at 183.515 110.49 0)
+			(effects
+				(font
+					(size 1.27 1.27)
+				)
+			)
+		)
+		(property "Footprint" ""
+			(at 181.61 106.68 0)
+			(effects
+				(font
+					(size 1.27 1.27)
+				)
+				(hide yes)
+			)
+		)
+		(property "Datasheet" ""
+			(at 181.61 106.68 0)
+			(effects
+				(font
+					(size 1.27 1.27)
+				)
+				(hide yes)
+			)
+		)
+		(property "Description" "Special symbol for telling ERC where power comes from"
+			(at 181.61 106.68 0)
+			(effects
+				(font
+					(size 1.27 1.27)
+				)
+				(hide yes)
+			)
+		)
+		(pin "1"
+		)
+		(instances
+			(project "RoyalBlue54L-Feather"
+				(path "/ba76ff89-c129-45ae-a3c9-97538370856c/0a43c989-a862-4ff1-8fb5-5f7c93f777a1"
+					(reference "#FLG05")
+					(unit 1)
+				)
