File: sch/Debugger.kicad_sch (KiCad schematic)
At the start: 29 parts, among them J3 USB_C_Receptacle_USB2.0_16P, J8 Conn_ARM_SWD_TagConnect_TC203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, U3 TPD3E001DRLR, U5 nRF52833-QDXX, U6 TXB0106RGY, Y2 32MHz

Commit message: Fix the Feather's ERC and DRC findings, without changing its rules
Modified Source of the RoyalBlue54L Feather by Helmut Lord (Lord's Boards),
under CERN-OHL-P v2, from 9177387. Made on 25 September 2026 by an AI agent
(Claude, by Anthropic) through the Eloom CLI, for Matrice Technologies.
CHANGES.md is the licence's modification notice and lists every change.

- PWR_FLAG on five externally fed nets (5 power_pin_not_driven errors)
- TP7 moved 0.049 mm onto the 1.27 mm grid (4 endpoint_off_grid warnings)
- four short reroutes for hole clearance (5 hole_clearance errors)
- courtyards: TP5-TP12 on 1.0 mm pads at the same pitch, J5 moved 0.32 mm,
  J3 and J5 courtyards drawn to their outlines, J2 on the back like J1 with a
  mirrored footprint and identical copper (11 courtyards_overlap errors)
- the design's own embedded symbols and footprints archived verbatim into
  project libraries; nothing updated from KiCad 10's libraries
- silkscreen nudges: the "+" mark, LOGO1, R5 and C9

The project file, with the author's rules and exclusions, is 9177387's byte
for byte. ERC 43 -> 0 and DRC 62 -> 0 with schematic parity, KiCad 10.0.6;
the final runs are under runs/. The author has not reviewed these changes,
and passing ERC and DRC does not prove the board works.

Co-Authored-By: Claude Opus 5.5 <noreply@anthropic.com>
Parts:
- C10, C15, C16, C17, C18, C19, C20, C21, C22, C23, C24, C25, C7: footprint Capacitor_SMD:C_0402_1005Metric -> RoyalBlue54L-Feather:C_0402_1005Metric; symbol Device:C_Small -> RoyalBlue54L-Feather:C_Small
- J3: footprint marbastlib-various:USB_C_Receptacle_HRO_TYPE-C-31-M-12 -> RoyalBlue54L-Feather:USB_C_Receptacle_HRO_TYPE-C-31-M-12_ChamferedCourtyard; symbol Connector:USB_C_Receptacle_USB2.0_16P -> RoyalBlue54L-Feather:USB_C_Receptacle_USB2.0_16P
- R1, R8: footprint Resistor_SMD:R_0402_1005Metric -> RoyalBlue54L-Feather:R_0402_1005Metric
- TP10, TP11, TP12, TP5, TP6, TP7, TP8, TP9: footprint TestPoint:TestPoint_Pad_D1.5mm -> TestPoint:TestPoint_Pad_D1.0mm
- U3: footprint Package_TO_SOT_SMD:SOT-553 -> RoyalBlue54L-Feather:SOT-553
- U5: footprint Package_DFN_QFN:QFN-40-1EP_5x5mm_P0.4mm_EP3.6x3.6mm_ThermalVias -> RoyalBlue54L-Feather:QFN-40-1EP_5x5mm_P0.4mm_EP3.6x3.6mm_ThermalVias; symbol nordic-lib-kicad-nrf52:nRF52833-QDXX -> RoyalBlue54L-Feather:nRF52833-QDXX
- Y2: footprint Crystal:Crystal_SMD_2016-4Pin_2.0x1.6mm -> RoyalBlue54L-Feather:Crystal_SMD_2016-4Pin_2.0x1.6mm; symbol hlord2000-Device:Crystal_GND24_Small_EZRoute -> RoyalBlue54L-Feather:Crystal_GND24_Small_EZRoute
