File: sch/nPM1300.kicad_sch (KiCad schematic)
At the start: 13 parts, among them U2 nPM1300-QEXX

Commit message: Fix the Feather's ERC and DRC findings, without changing its rules
Modified Source of the RoyalBlue54L Feather by Helmut Lord (Lord's Boards),
under CERN-OHL-P v2, from 9177387. Made on 25 September 2026 by an AI agent
(Claude, by Anthropic) through the Eloom CLI, for Matrice Technologies.
CHANGES.md is the licence's modification notice and lists every change.

- PWR_FLAG on five externally fed nets (5 power_pin_not_driven errors)
- TP7 moved 0.049 mm onto the 1.27 mm grid (4 endpoint_off_grid warnings)
- four short reroutes for hole clearance (5 hole_clearance errors)
- courtyards: TP5-TP12 on 1.0 mm pads at the same pitch, J5 moved 0.32 mm,
  J3 and J5 courtyards drawn to their outlines, J2 on the back like J1 with a
  mirrored footprint and identical copper (11 courtyards_overlap errors)
- the design's own embedded symbols and footprints archived verbatim into
  project libraries; nothing updated from KiCad 10's libraries
- silkscreen nudges: the "+" mark, LOGO1, R5 and C9

The project file, with the author's rules and exclusions, is 9177387's byte
for byte. ERC 43 -> 0 and DRC 62 -> 0 with schematic parity, KiCad 10.0.6;
the final runs are under runs/. The author has not reviewed these changes,
and passing ERC and DRC does not prove the board works.

Co-Authored-By: Claude Opus 5.5 <noreply@anthropic.com>
Parts:
- C1: footprint Capacitor_SMD:C_0402_1005Metric -> RoyalBlue54L-Feather:C_0402_1005Metric; symbol Device:C_Small -> RoyalBlue54L-Feather:C_Small
- C11, C2, C3, C4, C5, C6, C8: footprint Capacitor_SMD:C_0603_1608Metric -> RoyalBlue54L-Feather:C_0603_1608Metric; symbol Device:C_Small -> RoyalBlue54L-Feather:C_Small
- JP1: symbol Jumper:SolderJumper_2_Bridged -> RoyalBlue54L-Feather:SolderJumper_2_Bridged
- L1: footprint Inductor_SMD:L_0603_1608Metric -> RoyalBlue54L-Feather:L_0603_1608Metric
- R4: footprint Resistor_SMD:R_0402_1005Metric -> RoyalBlue54L-Feather:R_0402_1005Metric
- U2: footprint Package_DFN_QFN:QFN-32-1EP_5x5mm_P0.5mm_EP3.6x3.6mm_ThermalVias -> RoyalBlue54L-Feather:QFN-32-1EP_5x5mm_P0.5mm_EP3.6x3.6mm_ThermalVias; symbol nordic-lib-kicad-npm:nPM1300-QEXX -> RoyalBlue54L-Feather:nPM1300-QEXX
Changed lines of the file:
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@@
+		(color 0 0 0 0)
+	)
+	(junction
+		(at 231.14 93.98)
+		(diameter 0)
 		(color 0 0 0 0)
 	)
@@
 	(wire
 		(pts
-			(xy 234.95 93.98) (xy 228.6 93.98)
+			(xy 234.95 93.98) (xy 231.14 93.98)
+		)
+		(stroke
+			(width 0)
+			(type default)
+		)
+	)
+	(wire
+		(pts
+			(xy 231.14 93.98) (xy 228.6 93.98)
 		)
 		(stroke
@@
 	)
 	(symbol
-		(lib_id "Device:C_Small")
+		(lib_id "RoyalBlue54L-Feather:C_Small")
 		(at 194.31 132.08 0)
 		(mirror y)
@@
 			)
 		)
-		(property "Footprint" "Capacitor_SMD:C_0603_1608Metric"
+		(property "Footprint" "RoyalBlue54L-Feather:C_0603_1608Metric"
 			(at 194.31 132.08 0)
 			(effects
@@
 			)
 		)
-		(property "Footprint" "Inductor_SMD:L_0603_1608Metric"
+		(property "Footprint" "RoyalBlue54L-Feather:L_0603_1608Metric"
 			(at 203.2 96.52 0)
 			(effects
@@
 	)
 	(symbol
-		(lib_id "Device:C_Small")
+		(lib_id "RoyalBlue54L-Feather:C_Small")
 		(at 101.6 68.58 0)
 		(unit 1)
@@
 			)
 		)
-		(property "Footprint" "Capacitor_SMD:C_0603_1608Metric"
+		(property "Footprint" "RoyalBlue54L-Feather:C_0603_1608Metric"
 			(at 101.6 68.58 0)
 			(effects
@@
 	)
 	(symbol
-		(lib_id "Device:C_Small")
+		(lib_id "RoyalBlue54L-Feather:C_Small")
 		(at 214.63 96.52 0)
 		(mirror y)
@@
 			)
 		)
-		(property "Footprint" "Capacitor_SMD:C_0603_1608Metric"
+		(property "Footprint" "RoyalBlue54L-Feather:C_0603_1608Metric"
 			(at 214.63 96.52 0)
 			(effects
@@
 	)
 	(symbol
-		(lib_id "Device:C_Small")
+		(lib_id "RoyalBlue54L-Feather:C_Small")
 		(at 168.91 49.53 0)
 		(mirror y)
@@
 			)
 		)
-		(property "Footprint" "Capacitor_SMD:C_0603_1608Metric"
+		(property "Footprint" "RoyalBlue54L-Feather:C_0603_1608Metric"
 			(at 168.91 49.53 0)
 			(effects
@@
 	)
 	(symbol
-		(lib_id "Device:C_Small")
+		(lib_id "RoyalBlue54L-Feather:C_Small")
 		(at 179.07 49.53 0)
 		(mirror y)
@@
 			)
 		)
-		(property "Footprint" "Capacitor_SMD:C_0603_1608Metric"
+		(property "Footprint" "RoyalBlue54L-Feather:C_0603_1608Metric"
 			(at 179.07 49.53 0)
 			(effects
@@
 	)
 	(symbol
-		(lib_id "Device:C_Small")
+		(lib_id "RoyalBlue54L-Feather:C_Small")
 		(at 194.31 69.85 0)
 		(mirror y)
@@
 			)
 		)
-		(property "Footprint" "Capacitor_SMD:C_0603_1608Metric"
+		(property "Footprint" "RoyalBlue54L-Feather:C_0603_1608Metric"
 			(at 194.31 69.85 0)
 			(effects
@@
 	)
 	(symbol
-		(lib_id "Device:C_Small")
+		(lib_id "RoyalBlue54L-Feather:C_Small")
 		(at 158.75 49.53 0)
 		(mirror y)
@@
 			)
 		)
-		(property "Footprint" "Capacitor_SMD:C_0603_1608Metric"
+		(property "Footprint" "RoyalBlue54L-Feather:C_0603_1608Metric"
 			(at 158.75 49.53 0)
 			(effects
@@
 	)
 	(symbol
-		(lib_id "nordic-lib-kicad-npm:nPM1300-QEXX")
+		(lib_id "RoyalBlue54L-Feather:nPM1300-QEXX")
 		(at 148.59 99.06 0)
 		(unit 1)
@@
 			)
 		)
-		(property "Footprint" "Package_DFN_QFN:QFN-32-1EP_5x5mm_P0.5mm_EP3.6x3.6mm_ThermalVias"
+		(property "Footprint" "RoyalBlue54L-Feather:QFN-32-1EP_5x5mm_P0.5mm_EP3.6x3.6mm_ThermalVias"
 			(at 148.59 45.72 0)
 			(effects
@@
 	)
 	(symbol
-		(lib_id "Device:C_Small")
+		(lib_id "RoyalBlue54L-Feather:C_Small")
 		(at 140.97 49.53 0)
 		(unit 1)
@@
 			)
 		)
-		(property "Footprint" "Capacitor_SMD:C_0402_1005Metric"
+		(property "Footprint" "RoyalBlue54L-Feather:C_0402_1005Metric"
 			(at 140.97 49.53 0)
 			(effects
@@
 	)
 	(symbol
-		(lib_id "Jumper:SolderJumper_2_Bridged")
+		(lib_id "RoyalBlue54L-Feather:SolderJumper_2_Bridged")
 		(at 224.79 93.98 0)
 		(unit 1)
@@
 			)
 		)
-		(property "Footprint" "Resistor_SMD:R_0402_1005Metric"
+		(property "Footprint" "RoyalBlue54L-Feather:R_0402_1005Metric"
 			(at 100.33 124.46 0)
 			(effects
@@
 					(unit 1)
 				)
+			)
+		)
+	)
+	(symbol
+		(lib_id "power:PWR_FLAG")
+		(at 231.14 93.98 180)
+		(unit 1)
+		(exclude_from_sim no)
+		(in_bom yes)
+		(on_board yes)
+		(dnp no)
+		(property "Reference" "#FLG03"
+			(at 231.14 95.885 0)
+			(effects
+				(font
+					(size 1.27 1.27)
+				)
+				(hide yes)
+			)
+		)
+		(property "Value" "PWR_FLAG"
+			(at 231.14 97.79 0)
+			(effects
+				(font
+					(size 1.27 1.27)
+				)
+			)
+		)
+		(property "Footprint" ""
+			(at 231.14 93.98 0)
+			(effects
+				(font
+					(size 1.27 1.27)
+				)
+				(hide yes)
+			)
+		)
+		(property "Datasheet" ""
+			(at 231.14 93.98 0)
+			(effects
+				(font
+					(size 1.27 1.27)
+				)
+				(hide yes)
+			)
+		)
+		(property "Description" "Special symbol for telling ERC where power comes from"
+			(at 231.14 93.98 0)
+			(effects
+				(font
+					(size 1.27 1.27)
+				)
+				(hide yes)
+			)
+		)
+		(pin "1"
+		)
+		(instances
+			(project "RoyalBlue54L-Feather"
+				(path "/ba76ff89-c129-45ae-a3c9-97538370856c/79d06a01-15ae-4276-9cac-debde3b18a91"
+					(reference "#FLG03")
+					(unit 1)
+				)
