File: sch/nRF54L15.kicad_sch (KiCad schematic)
At the start: 18 parts, among them J6 Conn_01x05_MountingPin, SW1 SW_Push, SW2 SW_Push, U1 BM15x, U4 W25Q16JVUXIQ, Y1 32.768KHz

Commit message: Fix the Feather's ERC and DRC findings, without changing its rules
Modified Source of the RoyalBlue54L Feather by Helmut Lord (Lord's Boards),
under CERN-OHL-P v2, from 9177387. Made on 25 September 2026 by an AI agent
(Claude, by Anthropic) through the Eloom CLI, for Matrice Technologies.
CHANGES.md is the licence's modification notice and lists every change.

- PWR_FLAG on five externally fed nets (5 power_pin_not_driven errors)
- TP7 moved 0.049 mm onto the 1.27 mm grid (4 endpoint_off_grid warnings)
- four short reroutes for hole clearance (5 hole_clearance errors)
- courtyards: TP5-TP12 on 1.0 mm pads at the same pitch, J5 moved 0.32 mm,
  J3 and J5 courtyards drawn to their outlines, J2 on the back like J1 with a
  mirrored footprint and identical copper (11 courtyards_overlap errors)
- the design's own embedded symbols and footprints archived verbatim into
  project libraries; nothing updated from KiCad 10's libraries
- silkscreen nudges: the "+" mark, LOGO1, R5 and C9

The project file, with the author's rules and exclusions, is 9177387's byte
for byte. ERC 43 -> 0 and DRC 62 -> 0 with schematic parity, KiCad 10.0.6;
the final runs are under runs/. The author has not reviewed these changes,
and passing ERC and DRC does not prove the board works.

Co-Authored-By: Claude Opus 5.5 <noreply@anthropic.com>
Parts:
- C12, C13, C14, C9: footprint Capacitor_SMD:C_0402_1005Metric -> RoyalBlue54L-Feather:C_0402_1005Metric; symbol Device:C_Small -> RoyalBlue54L-Feather:C_Small
- D1: footprint LED_SMD:LED_0603_1608Metric -> RoyalBlue54L-Feather:LED_0603_1608Metric; symbol Device:LED_Small -> RoyalBlue54L-Feather:LED_Small
- R5, R6, R7: footprint Resistor_SMD:R_0402_1005Metric -> RoyalBlue54L-Feather:R_0402_1005Metric
- U1: footprint nordic-lib-kicad-nrf54-modules:BM15x-LGA-45_15.8x10mm -> RoyalBlue54L-Feather:BM15x-LGA-45_15.8x10mm; symbol nordic-lib-kicad-nrf54-modules:BM15x -> RoyalBlue54L-Feather:BM15x
- U4: footprint Package_SON:Winbond_USON-8-1EP_3x2mm_P0.5mm_EP0.2x1.6mm -> RoyalBlue54L-Feather:Winbond_USON-8-1EP_3x2mm_P0.5mm_EP0.2x1.6mm
Changed lines of the file:
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@@
 	)
 	(symbol
-		(lib_id "Device:LED_Small")
+		(lib_id "RoyalBlue54L-Feather:LED_Small")
 		(at 93.98 115.57 270)
 		(mirror x)
@@
 			)
 		)
-		(property "Footprint" "LED_SMD:LED_0603_1608Metric"
+		(property "Footprint" "RoyalBlue54L-Feather:LED_0603_1608Metric"
 			(at 93.98 115.57 90)
 			(effects
@@
 			)
 		)
-		(property "Footprint" "Package_SON:Winbond_USON-8-1EP_3x2mm_P0.5mm_EP0.2x1.6mm"
+		(property "Footprint" "RoyalBlue54L-Feather:Winbond_USON-8-1EP_3x2mm_P0.5mm_EP0.2x1.6mm"
 			(at 63.5 105.41 0)
 			(effects
@@
 			)
 		)
-		(property "Footprint" "Resistor_SMD:R_0402_1005Metric"
+		(property "Footprint" "RoyalBlue54L-Feather:R_0402_1005Metric"
 			(at 179.07 62.23 0)
 			(effects
@@
 	)
 	(symbol
-		(lib_id "nordic-lib-kicad-nrf54-modules:BM15x")
+		(lib_id "RoyalBlue54L-Feather:BM15x")
 		(at 137.16 90.17 0)
 		(unit 1)
@@
 			)
 		)
-		(property "Footprint" "nordic-lib-kicad-nrf54-modules:BM15x-LGA-45_15.8x10mm"
+		(property "Footprint" "RoyalBlue54L-Feather:BM15x-LGA-45_15.8x10mm"
 			(at 137.16 90.17 0)
 			(effects
@@
 			)
 		)
-		(property "Footprint" "Resistor_SMD:R_0402_1005Metric"
+		(property "Footprint" "RoyalBlue54L-Feather:R_0402_1005Metric"
 			(at 181.61 62.23 0)
 			(effects
@@
 	)
 	(symbol
-		(lib_id "Device:C_Small")
+		(lib_id "RoyalBlue54L-Feather:C_Small")
 		(at 83.82 67.31 0)
 		(mirror y)
@@
 			)
 		)
-		(property "Footprint" "Capacitor_SMD:C_0402_1005Metric"
+		(property "Footprint" "RoyalBlue54L-Feather:C_0402_1005Metric"
 			(at 83.82 67.31 0)
 			(effects
@@
 	)
 	(symbol
-		(lib_id "Device:C_Small")
+		(lib_id "RoyalBlue54L-Feather:C_Small")
 		(at 132.08 45.72 0)
 		(mirror y)
@@
 			)
 		)
-		(property "Footprint" "Capacitor_SMD:C_0402_1005Metric"
+		(property "Footprint" "RoyalBlue54L-Feather:C_0402_1005Metric"
 			(at 132.08 45.72 0)
 			(effects
@@
 	)
 	(symbol
-		(lib_id "Device:C_Small")
+		(lib_id "RoyalBlue54L-Feather:C_Small")
 		(at 57.15 82.55 0)
 		(unit 1)
@@
 			)
 		)
-		(property "Footprint" "Capacitor_SMD:C_0402_1005Metric"
+		(property "Footprint" "RoyalBlue54L-Feather:C_0402_1005Metric"
 			(at 57.15 82.55 0)
 			(effects
@@
 			)
 		)
-		(property "Footprint" "Resistor_SMD:R_0402_1005Metric"
+		(property "Footprint" "RoyalBlue54L-Feather:R_0402_1005Metric"
 			(at 93.98 120.65 0)
 			(effects
@@
 	)
 	(symbol
-		(lib_id "Device:C_Small")
+		(lib_id "RoyalBlue54L-Feather:C_Small")
 		(at 96.52 64.77 0)
 		(mirror y)
@@
 			)
 		)
-		(property "Footprint" "Capacitor_SMD:C_0402_1005Metric"
+		(property "Footprint" "RoyalBlue54L-Feather:C_0402_1005Metric"
 			(at 96.52 64.77 0)
 			(effects
